Commit message: gazebo model in the air

File: urdf/uniped.xacro (robot description, xacro)
@@ -15,4 +15,5 @@
   <xacro:property name="foot_width" value="0.3" /> <!-- width of the foot -->
   <xacro:property name="foot_length" value="0.3" /> <!-- length of the foot -->
+  <xacro:property name="height" value="1" /> <!-- height of the robot in the air -->
   <xacro:property name="gravity_off" value="1" /> <!-- use gravity flag -->
   <!-- Import all Gazebo-customization elements, including Gazebo colors -->
@@ -23,5 +24,5 @@
   <link name="torso">
     <collision>
-      <origin xyz="0 0 ${torso_length/2 + tigh_length + calf_length + foot_height}" rpy="0 0 0"/>
+      <origin xyz="0 0 ${torso_length/2 + tigh_length + calf_length + foot_height + height}" rpy="0 0 0"/>
       <geometry>
 	<box size="${torso_width} ${torso_thickness} ${torso_length}"/>
@@ -29,5 +30,5 @@
     </collision>
     <visual>
-      <origin xyz="0 0 ${torso_length/2 + tigh_length + calf_length + foot_height}" rpy="0 0 0"/>
+      <origin xyz="0 0 ${torso_length/2 + tigh_length + calf_length + foot_height + height}" rpy="0 0 0"/>
       <geometry>
 	     <box size="${torso_width} ${torso_thickness} ${torso_length}"/>
@@ -36,5 +37,5 @@
     </visual>
     <inertial>
-      <origin xyz="0 0 ${torso_length/2 + tigh_length + calf_length + foot_height}" rpy="0 0 0"/>
+      <origin xyz="0 0 ${torso_length/2 + tigh_length + calf_length + foot_height + height}" rpy="0 0 0"/>
       <mass value="${mass}"/>
       <inertia
@@ -47,5 +48,5 @@
     <parent link="torso"/>
     <child link="tigh"/>
-    <origin xyz="0 0 ${tigh_length + calf_length + foot_height}" rpy="0 0 0"/>
+    <origin xyz="0 0 ${tigh_length + calf_length + foot_height + height}" rpy="0 0 0"/>
     <axis xyz="1 0 0"/>
     <dynamics damping="0.7"/>

Commit message: removed damping

File: urdf/uniped.xacro (robot description, xacro)
@@ -50,5 +50,5 @@
     <origin xyz="0 0 ${tigh_length + calf_length + foot_height + height}" rpy="0 0 0"/>
     <axis xyz="1 0 0"/>
-    <dynamics damping="0.7"/>
+    <dynamics damping="0.0"/>
   </joint>
   <!-- Tigh Link -->
@@ -81,5 +81,5 @@
     <origin xyz="0 0 ${- tigh_length}" rpy="0 0 0"/>
     <axis xyz="1 0 0"/>
-    <dynamics damping="0.7"/>
+    <dynamics damping="0.0"/>
   </joint>
   <link name="calf">
@@ -111,5 +111,5 @@
     <origin xyz="0 0 ${- calf_length}" rpy="0 0 0"/>
     <axis xyz="1 0 0"/>
-    <dynamics damping="0.7"/>
+    <dynamics damping="0.0"/>
   </joint>
   <link name="foot">
